Commit message: feat(mapping,nav,urdf): add 2D/3D SLAM modes, map export scripts, autonomous nav bringup and updated URDF architecture

File: src/hoverboard_base/urdf/robot.urdf (robot description, URDF)
Before this commit: robot hoverboard_robot, 6 links, 5 joints
Links:
- added link camera_link; collision box size=0.025 0.090 0.025; visual box size=0.025 0.090 0.025
- added link pan_link; collision box size=0.045 0.045 0.05; visual box size=0.045 0.045 0.05
- added link pan_tilt_base_link; collision cylinder length=0.03 radius=0.035; visual cylinder length=0.03 radius=0.035
- added link tilt_link; collision box size=0.04 0.10 0.03; visual box size=0.04 0.10 0.03
- added link torso_column, mass 3.5; collision box size=0.06 0.06 1.0; visual box size=0.06 0.06 1.0
- added link torso_lift_link; collision box size=0.10 0.12 0.02; visual box size=0.10 0.12 0.02
Joints:
- added joint camera_mount_joint: type fixed, parent tilt_link, child camera_link, origin xyz=0.035 0.0 0.015 rpy=0 0 0
- added joint pan_joint: type revolute, parent pan_tilt_base_link, child pan_link, origin xyz=0 0 0.03 rpy=0 0 0, axis 0 0 1, limit lower=-1.5708 upper=1.5708 effort=2.5 velocity=3.14
- added joint pan_tilt_base_joint: type fixed, parent torso_lift_link, child pan_tilt_base_link, origin xyz=0 0 0.01 rpy=0 0 0
- added joint tilt_joint: type revolute, parent pan_link, child tilt_link, origin xyz=0 0 0.05 rpy=0 0 0, axis 0 1 0, limit lower=-0.7854 upper=0.7854 effort=2.5 velocity=3.14
- added joint torso_column_joint: type fixed, parent base_link, child torso_column, origin xyz=0.0 0.0 0.09 rpy=0 0 0
- added joint torso_lift_joint: type fixed, parent torso_column, child torso_lift_link, origin xyz=0 0 1.0 rpy=0 0 0

File: src/hoverboard_base/urdf/robot.urdf.xacro (robot description, xacro)
@@ -18,4 +18,9 @@
   <xacro:property name="laser_offset_y" value="0.00"/>
   <xacro:property name="laser_offset_z" value="0.18"/>
+  <!-- Sistema de Elevación Torso / Columna (Exactamente en el medio de la base, 1.0 m altura) -->
+  <xacro:property name="column_x"       value="0.0"/>
+  <xacro:property name="column_y"       value="0.0"/>
+  <xacro:property name="column_height"  value="1.0"/>
+  <xacro:property name="column_width"   value="0.06"/>
   <!-- ==================== MATERIALES ==================== -->
   <material name="chassis_blue">
@@ -30,4 +35,13 @@
   <material name="caster_gray">
     <color rgba="0.35 0.35 0.35 1.0"/>
+  </material>
+  <material name="column_aluminum">
+    <color rgba="0.65 0.65 0.70 1.0"/>
+  </material>
+  <material name="pantilt_dark">
+    <color rgba="0.18 0.18 0.18 1.0"/>
+  </material>
+  <material name="realsense_silver">
+    <color rgba="0.75 0.75 0.75 1.0"/>
   </material>
   <!-- ==================== BASE FOOTPRINT ==================== -->
@@ -127,3 +141,142 @@
     <origin xyz="${laser_offset_x} ${laser_offset_y} ${laser_offset_z}" rpy="0 0 0"/>
   </joint>
+  <!-- ==================== SISTEMA DE SUBIR Y BAJAR (TORSO VERTICAL) ==================== -->
+  <!-- Columna estructural fija exactamente en el medio de la base (x=0, y=0) con 1 metro de altura -->
+  <link name="torso_column">
+    <visual>
+      <origin xyz="0 0 ${column_height / 2.0}" rpy="0 0 0"/>
+      <geometry>
+        <box size="${column_width} ${column_width} ${column_height}"/>
+      </geometry>
+      <material name="column_aluminum"/>
+    </visual>
+    <collision>
+      <origin xyz="0 0 ${column_height / 2.0}" rpy="0 0 0"/>
+      <geometry>
+        <box size="${column_width} ${column_width} ${column_height}"/>
+      </geometry>
+    </collision>
+    <inertial>
+      <origin xyz="0 0 ${column_height / 2.0}" rpy="0 0 0"/>
+      <mass value="3.5"/>
+      <inertia ixx="0.292" ixy="0.0" ixz="0.0" iyy="0.292" iyz="0.0" izz="0.002"/>
+    </inertial>
+  </link>
+  <joint name="torso_column_joint" type="fixed">
+    <parent link="base_link"/>
+    <child link="torso_column"/>
+    <origin xyz="${column_x} ${column_y} ${ground_clearance + chassis_height}" rpy="0 0 0"/>
+  </joint>
+  <!-- Plataforma superior móvil del elevador (a 1.0 m arriba en la parte superior) -->
+  <link name="torso_lift_link">
+    <visual>
+      <origin xyz="0 0 0" rpy="0 0 0"/>
+      <geometry>
+        <box size="0.10 0.12 0.02"/>
+      </geometry>
+      <material name="pantilt_dark"/>
+    </visual>
+    <collision>
+      <origin xyz="0 0 0" rpy="0 0 0"/>
+      <geometry>
+        <box size="0.10 0.12 0.02"/>
+      </geometry>
+    </collision>
+  </link>
+  <!-- Joint de elevación / tope superior de columna (fijo a 1.0 m de altura) -->
+  <joint name="torso_lift_joint" type="fixed">
+    <parent link="torso_column"/>
+    <child link="torso_lift_link"/>
+    <origin xyz="0 0 ${column_height}" rpy="0 0 0"/>
+  </joint>
+  <!-- ==================== SISTEMA PAN-TILT ==================== -->
+  <!-- Base de montaje del Pan-Tilt -->
+  <link name="pan_tilt_base_link">
+    <visual>
+      <origin xyz="0 0 0.015" rpy="0 0 0"/>
+      <geometry>
+        <cylinder radius="0.035" length="0.03"/>
+      </geometry>
+      <material name="pantilt_dark"/>
+    </visual>
+    <collision>
+      <origin xyz="0 0 0.015" rpy="0 0 0"/>
+      <geometry>
+        <cylinder radius="0.035" length="0.03"/>
+      </geometry>
+    </collision>
+  </link>
+  <joint name="pan_tilt_base_joint" type="fixed">
+    <parent link="torso_lift_link"/>
+    <child link="pan_tilt_base_link"/>
+    <origin xyz="0 0 0.01" rpy="0 0 0"/>
+  </joint>
+  <!-- Motor 1: Pan Joint (Giro Horizontal en Z) -->
+  <link name="pan_link">
+    <visual>
+      <origin xyz="0 0 0.025" rpy="0 0 0"/>
+      <geometry>
+        <box size="0.045 0.045 0.05"/>
+      </geometry>
+      <material name="pantilt_dark"/>
+    </visual>
+    <collision>
+      <origin xyz="0 0 0.025" rpy="0 0 0"/>
+      <geometry>
+        <box size="0.045 0.045 0.05"/>
+      </geometry>
+    </collision>
+  </link>
+  <joint name="pan_joint" type="revolute">
+    <parent link="pan_tilt_base_link"/>
+    <child link="pan_link"/>
+    <origin xyz="0 0 0.03" rpy="0 0 0"/>
+    <axis xyz="0 0 1"/>
+    <limit lower="-1.5708" upper="1.5708" effort="2.5" velocity="3.14"/>
+  </joint>
+  <!-- Motor 2: Tilt Joint (Inclinación Vertical en Y) -->
+  <link name="tilt_link">
+    <visual>
+      <origin xyz="0.015 0 0.01" rpy="0 0 0"/>
+      <geometry>
+        <box size="0.04 0.10 0.03"/>
+      </geometry>
+      <material name="pantilt_dark"/>
+    </visual>
+    <collision>
+      <origin xyz="0.015 0 0.01" rpy="0 0 0"/>
+      <geometry>
+        <box size="0.04 0.10 0.03"/>
+      </geometry>
+    </collision>
+  </link>
+  <joint name="tilt_joint" type="revolute">
+    <parent link="pan_link"/>
+    <child link="tilt_link"/>
+    <origin xyz="0 0 0.05" rpy="0 0 0"/>
+    <axis xyz="0 1 0"/>
+    <limit lower="-0.7854" upper="0.7854" effort="2.5" velocity="3.14"/>
+  </joint>
+  <!-- ==================== CÁMARA INTEL REALSENSE D435 ==================== -->
+  <!-- Conexión rígida entre el soporte tilt y el marco base de la RealSense (camera_link) -->
+  <joint name="camera_mount_joint" type="fixed">
+    <parent link="tilt_link"/>
+    <child link="camera_link"/>
+    <origin xyz="0.035 0.0 0.015" rpy="0 0 0"/>
+  </joint>
+  <link name="camera_link">
+    <visual>
+      <origin xyz="0 0 0" rpy="0 0 0"/>
+      <geometry>
+        <box size="0.025 0.090 0.025"/>
+      </geometry>
+      <material name="realsense_silver"/>
+    </visual>
+    <collision>
+      <origin xyz="0 0 0" rpy="0 0 0"/>
+      <geometry>
+        <box size="0.025 0.090 0.025"/>
+      </geometry>
+    </collision>
+  </link>
 </robot>

Commit message: feat(manipulation): implement 3-phase autonomous grasping, lead-through teaching for home/pre-grasp, and complete Piper URDF
- Add unified master manipulation script 'manipulacion_autonoma.py' with 3 operational phases:
  * Phase 1: Safe movement envelope & hard-stop interlock monitor
  * Phase 2: Stowed/Home pose execution and manual lead-through teaching
  * Phase 3: Pre-grasp positioning, manual lead-through teaching, and 5-stage autonomous cycle
- Add lead-through manual teaching mode for both Home and Pre-Grasp with live torque release and YAML persistence
- Fix Pan-Tilt inverted controls (W tilts up, S tilts down, A pans left, D pans right, T aims at table)
- Integrate PiperKinematicsSolver with weighted DLS IK, nullspace roll stabilization, and camera-to-arm 3D transformation
- Update robot URDF/Xacro with elevator carriage, 35x25cm mounting prism (12cm below pan-tilt), left-mounted Piper arm, and DaBai eye-in-hand camera link
- Add Piper meshes, descriptions, and custom ROS 2 message definitions
- Back up Jetson Orin Nano controller scripts in scripts/jetson/

File: src/hoverboard_base/urdf/robot.urdf (robot description, URDF)
Before this commit: robot hoverboard_robot, 12 links, 11 joints
Links:
- added link arm_base_link, mass 1.02; collision mesh filename=package://piper_description/meshes/base_link.STL; visual mesh filename=package://piper_description/meshes/base_link.STL
- added link arm_camera_link, mass 0.08; collision box size=0.030 0.090 0.025; visual box size=0.030 0.090 0.025
- added link arm_camera_optical_frame
- added link camera_color_optical_frame
- added link gripper_base, mass 0.15; collision mesh filename=package://piper_description/meshes/gripper_base.STL; visual mesh filename=package://piper_description/meshes/gripper_base.STL
- added link link1, mass 0.71; collision mesh filename=package://piper_description/meshes/link1.STL; visual mesh filename=package://piper_description/meshes/link1.STL
- added link link2, mass 1.16; collision mesh filename=package://piper_description/meshes/link2.STL; visual mesh filename=package://piper_description/meshes/link2.STL
- added link link3, mass 0.71; collision mesh filename=package://piper_description/meshes/link3.STL; visual mesh filename=package://piper_description/meshes/link3.STL
- added link link4, mass 0.27; collision mesh filename=package://piper_description/meshes/link4.STL; visual mesh filename=package://piper_description/meshes/link4.STL
- added link link5, mass 0.4; collision mesh filename=package://piper_description/meshes/link5.STL; visual mesh filename=package://piper_description/meshes/link5.STL
- added link link6, mass 0.21; collision mesh filename=package://piper_description/meshes/link6.STL; visual mesh filename=package://piper_description/meshes/link6.STL
- added link link7, mass 0.025; collision mesh filename=package://piper_description/meshes/link7.STL; visual mesh filename=package://piper_description/meshes/link7.STL
- added link link8, mass 0.025; collision mesh filename=package://piper_description/meshes/link8.STL; visual mesh filename=package://piper_description/meshes/link8.STL
- added link mounting_cube_link, mass 4.0; collision box size=0.25 0.35 0.35; visual box size=0.25 0.35 0.35
- added link screen_link, mass 1.2; collision box size=0.05 0.27 0.19; visual box size=0.002 0.24000000000000002 0.16
- link camera_link: mass None -> 0.072
- link pan_link: mass None -> 0.15
- link pan_tilt_base_link: mass None -> 0.25
- link tilt_link: mass None -> 0.15
- link torso_column: geometry collision box size=0.08 0.08 1.0; visual box size=0.06 0.06 1.0
- link torso_lift_link: mass None -> 1.8; geometry collision box size=0.22 0.38 0.02; visual box size=0.22 0.38 0.02
Joints:
- added joint arm_camera_mount_joint: type fixed, parent gripper_base, child arm_camera_link, origin xyz=0.025 0.0 0.08 rpy=0 0 0
- added joint arm_camera_optical_joint: type fixed, parent arm_camera_link, child arm_camera_optical_frame, origin xyz=0 0 0 rpy=-1.5707963 0 -1.5707963
- added joint camera_color_optical_joint: type fixed, parent camera_link, child camera_color_optical_frame, origin xyz=0 0 0 rpy=-1.5707963 0 -1.5707963
- added joint cube_to_arm_joint: type fixed, parent mounting_cube_link, child arm_base_link, origin xyz=0.0 0.175 0.10 rpy=-1.5707963 0 0
- added joint joint1: type revolute, parent arm_base_link, child link1, origin xyz=0 0 0.123 rpy=0 0 0, axis 0 0 1, limit lower=-2.618 upper=2.618 effort=100 velocity=5
- added joint joint2: type revolute, parent link1, child link2, origin xyz=0 0 0 rpy=0.785398 0 0, axis 0 1 0, limit lower=0 upper=3.1416 effort=100 velocity=5
- added joint joint3: type revolute, parent link2, child link3, origin xyz=0.265 0 0 rpy=-0.785398 0 0, axis 0 1 0, limit lower=-2.967 upper=0 effort=100 velocity=5
- added joint joint4: type revolute, parent link3, child link4, origin xyz=0.095 0 0 rpy=0 0 0, axis 1 0 0, limit lower=-1.745 upper=1.745 effort=100 velocity=5
- added joint joint5: type revolute, parent link4, child link5, origin xyz=0 0 0.123 rpy=0 0 0, axis 0 1 0, limit lower=-1.22 upper=1.22 effort=100 velocity=5
- added joint joint6: type revolute, parent link5, child link6, origin xyz=0.076 0 0 rpy=0 0 0, axis 1 0 0, limit lower=-2.094 upper=2.094 effort=100 velocity=5
- added joint joint6_to_gripper_base: type fixed, parent link6, child gripper_base, origin xyz=0 0 0 rpy=0 0 0
- added joint joint7: type prismatic, parent gripper_base, child link7, origin xyz=0 0 0.1358 rpy=1.5708 0 0, axis 0 0 1, limit lower=0 upper=0.035 effort=10 velocity=1
- added joint joint8: type prismatic, parent gripper_base, child link8, origin xyz=0 0 0.1358 rpy=1.5708 0 -3.1416, axis 0 0 -1, limit lower=-0.035 upper=0 effort=10 velocity=1
- added joint torso_lift_to_cube_joint: type fixed, parent torso_lift_link, child mounting_cube_link, origin xyz=0.155 0.0 -0.175 rpy=0 0 0
- added joint torso_lift_to_screen_joint: type fixed, parent torso_lift_link, child screen_link, origin xyz=0.30000000000000004 0.0 -0.175 rpy=0 0 0
- joint pan_tilt_base_joint: origin xyz=0 0 0.01 rpy=0 0 0 -> xyz=0.07 0.0 0.12 rpy=0 0 0

Commit message: Fix Piper 6-DOF official DH kinematics, side-mount Rx(-90) transform, RViz URDF meshes/axes, and CHARMIE Pre-Grasp seeded tool-line approach

File: src/hoverboard_base/urdf/robot.urdf (robot description, URDF)
Before this commit: robot robot_athome, 27 links, 26 joints
Links:
- added link tcp_link
- link link3: mass 0.71 -> 0.5
- link link4: mass 0.27 -> 0.38
- link link5: mass 0.4 -> 0.383
- link link6: mass 0.21 -> 0.007
Joints:
- added joint link6_to_tcp_joint: type fixed, parent link6, child tcp_link, origin xyz=0 0 0.1358 rpy=0 0 0
- joint joint1: limit lower=-2.618 upper=2.618 effort=100 velocity=5 -> lower=-2.688 upper=2.688 effort=100 velocity=5
- joint joint2: axis 0 1 0 -> 0 0 1; limit lower=0 upper=3.1416 effort=100 velocity=5 -> lower=0 upper=3.403 effort=100 velocity=5; origin xyz=0 0 0 rpy=0.785398 0 0 -> xyz=0 0 0 rpy=1.5708 -0.1359 -3.1416
- joint joint3: axis 0 1 0 -> 0 0 1; limit lower=-2.967 upper=0 effort=100 velocity=5 -> lower=-3.054 upper=0 effort=100 velocity=5; origin xyz=0.265 0 0 rpy=-0.785398 0 0 -> xyz=0.28503 0 0 rpy=0 0 -1.7939
- joint joint4: axis 1 0 0 -> 0 0 1; limit lower=-1.745 upper=1.745 effort=100 velocity=5 -> lower=-1.920 upper=1.920 effort=100 velocity=5; origin xyz=0.095 0 0 rpy=0 0 0 -> xyz=-0.021984 -0.25075 0 rpy=1.5708 0 0
- joint joint5: axis 0 1 0 -> 0 0 1; limit lower=-1.22 upper=1.22 effort=100 velocity=5 -> lower=-1.396 upper=1.396 effort=100 velocity=5; origin xyz=0 0 0.123 rpy=0 0 0 -> xyz=0 0 0 rpy=-1.5708 0 0
- joint joint6: axis 1 0 0 -> 0 0 1; limit lower=-2.094 upper=2.094 effort=100 velocity=5 -> lower=-3.142 upper=3.142 effort=100 velocity=3; origin xyz=0.076 0 0 rpy=0 0 0 -> xyz=8.8259E-05 -0.091 0 rpy=1.5708 0 0
- joint left_wheel_joint: axis 0 1 0 -> (none); type continuous -> fixed
- joint right_wheel_joint: axis 0 1 0 -> (none); type continuous -> fixed

File: src/hoverboard_base/urdf/robot_piper.urdf.xacro (robot description, xacro)
@@ -130,9 +130,8 @@
       </collision>
     </link>
-    <joint name="${prefix}_wheel_joint" type="continuous">
+    <joint name="${prefix}_wheel_joint" type="fixed">
       <parent link="base_link"/>
       <child link="${prefix}_wheel"/>
       <origin xyz="${wheel_offset_x} ${y_reflect * track_width / 2.0} ${wheel_radius}" rpy="0 0 0"/>
-      <axis xyz="0 1 0"/>
     </joint>
   </xacro:macro>
@@ -469,5 +468,5 @@
     <child link="link1" />
     <axis xyz="0 0 1" />
-    <limit lower="-2.618" upper="2.618" effort="100" velocity="5" />
+    <limit lower="-2.688" upper="2.688" effort="100" velocity="5" />
   </joint>
   <!-- Link 2 (Joint 2 - Hombro en Y) -->
@@ -493,16 +492,16 @@
   </link>
   <joint name="joint2" type="revolute">
-    <origin xyz="0 0 0" rpy="0.785398 0 0" />
+    <origin xyz="0 0 0" rpy="1.5708 -0.1359 -3.1416" />
     <parent link="link1" />
     <child link="link2" />
-    <axis xyz="0 1 0" />
-    <limit lower="0" upper="3.1416" effort="100" velocity="5" />
-  </joint>
-  <!-- Link 3 (Joint 3 - Codo en Y) -->
+    <axis xyz="0 0 1" />
+    <limit lower="0" upper="3.403" effort="100" velocity="5" />
+  </joint>
+  <!-- Link 3 (Joint 3 - Codo) -->
   <link name="link3">
     <inertial>
-      <origin xyz="0.08882 0.00142 -0.00494" rpy="0 0 0" />
-      <mass value="0.71" />
-      <inertia ixx="0.0003" ixy="0.0" ixz="0.0" iyy="0.011" iyz="0.0" izz="0.011" />
+      <origin xyz="-0.01999 -0.14808 -0.00053" rpy="0 0 0" />
+      <mass value="0.5" />
+      <inertia ixx="0.01347608" ixy="0.00161034" ixz="0.00000066" iyy="0.00046377" iyz="0.00000162" izz="0.01363321" />
     </inertial>
     <visual>
@@ -521,16 +520,16 @@
   </link>
   <joint name="joint3" type="revolute">
-    <origin xyz="0.265 0 0" rpy="-0.785398 0 0" />
+    <origin xyz="0.28503 0 0" rpy="0 0 -1.7939" />
     <parent link="link2" />
     <child link="link3" />
-    <axis xyz="0 1 0" />
-    <limit lower="-2.967" upper="0" effort="100" velocity="5" />
-  </joint>
-  <!-- Link 4 (Joint 4 - Giro Muñeca en X) -->
+    <axis xyz="0 0 1" />
+    <limit lower="-3.054" upper="0" effort="100" velocity="5" />
+  </joint>
+  <!-- Link 4 (Joint 4 - Muñeca Roll) -->
   <link name="link4">
     <inertial>
-      <origin xyz="-0.00017 -0.00845 0.03859" rpy="0 0 0" />
-      <mass value="0.27" />
-      <inertia ixx="0.0002" ixy="0.0" ixz="0.0" iyy="0.0002" iyz="0.0" izz="0.0001" />
+      <origin xyz="0.00013 -0.00076 -0.00394" rpy="0 0 0" />
+      <mass value="0.38" />
+      <inertia ixx="0.00017844" ixy="0.00000062" ixz="0.00000067" iyy="0.00018914" iyz="0.00000408" izz="0.00014613" />
     </inertial>
     <visual>
@@ -549,16 +548,16 @@
   </link>
   <joint name="joint4" type="revolute">
-    <origin xyz="0.095 0 0" rpy="0 0 0" />
+    <origin xyz="-0.021984 -0.25075 0" rpy="1.5708 0 0" />
     <parent link="link3" />
     <child link="link4" />
-    <axis xyz="1 0 0" />
-    <limit lower="-1.745" upper="1.745" effort="100" velocity="5" />
-  </joint>
-  <!-- Link 5 (Joint 5 - Cabeceo Muñeca en Y) -->
+    <axis xyz="0 0 1" />
+    <limit lower="-1.920" upper="1.920" effort="100" velocity="5" />
+  </joint>
+  <!-- Link 5 (Joint 5 - Muñeca Pitch) -->
   <link name="link5">
     <inertial>
-      <origin xyz="0.06078 0.00011 0.00015" rpy="0 0 0" />
-      <mass value="0.4" />
-      <inertia ixx="0.0001" ixy="0.0" ixz="0.0" iyy="0.0005" iyz="0.0" izz="0.0005" />
+      <origin xyz="0.00018 -0.06104 -0.00227" rpy="0 0 0" />
+      <mass value="0.383" />
+      <inertia ixx="0.00172318" ixy="0.00000259" ixz="0.00000010" iyy="0.00017936" iyz="0.00000990" izz="0.00171172" />
     </inertial>
     <visual>
@@ -577,16 +576,16 @@
   </link>
   <joint name="joint5" type="revolute">
-    <origin xyz="0 0 0.123" rpy="0 0 0" />
+    <origin xyz="0 0 0" rpy="-1.5708 0 0" />
     <parent link="link4" />
     <child link="link5" />
-    <axis xyz="0 1 0" />
-    <limit lower="-1.22" upper="1.22" effort="100" velocity="5" />
-  </joint>
-  <!-- Link 6 (Joint 6 - Giro Extremo Muñeca en Z) -->
+    <axis xyz="0 0 1" />
+    <limit lower="-1.396" upper="1.396" effort="100" velocity="5" />
+  </joint>
+  <!-- Link 6 (Joint 6 - Giro Extremo Muñeca) -->
   <link name="link6">
     <inertial>
-      <origin xyz="0.00011 0.00045 0.04022" rpy="0 0 0" />
-      <mass value="0.21" />
-      <inertia ixx="0.0001" ixy="0.0" ixz="0.0" iyy="0.0001" iyz="0.0" izz="0.0001" />
+      <origin xyz="-0.00003 0.00006 0.04618" rpy="0 0 0" />
+      <mass value="0.007" />
+      <inertia ixx="0.00152112" ixy="0.00000202" ixz="0.00000261" iyy="0.00138626" iyz="0.00000002" izz="0.00031152" />
     </inertial>
     <visual>
@@ -605,9 +604,16 @@
   </link>
   <joint name="joint6" type="revolute">
-    <origin xyz="0.076 0 0" rpy="0 0 0" />
+    <origin xyz="8.8259E-05 -0.091 0" rpy="1.5708 0 0" />
     <parent link="link5" />
     <child link="link6" />
-    <axis xyz="1 0 0" />
-    <limit lower="-2.094" upper="2.094" effort="100" velocity="5" />
+    <axis xyz="0 0 1" />
+    <limit lower="-3.142" upper="3.142" effort="100" velocity="3" />
+  </joint>
+  <!-- Punto Central de Herramienta (TCP) entre los dedos de la pinza -->
+  <link name="tcp_link"/>
+  <joint name="link6_to_tcp_joint" type="fixed">
+    <origin xyz="0 0 0.1358" rpy="0 0 0" />
+    <parent link="link6" />
+    <child link="tcp_link" />
   </joint>
   <!-- Pinza Paralela: Base de la Pinza -->

Commit message: Calibrate 6cm rightward wrist camera offset and full forward IK reach (+12-15.5cm) from Pre-Grasp

File: src/hoverboard_base/urdf/robot.urdf (robot description, URDF)
Before this commit: robot robot_athome, 28 links, 27 joints
Joints:
- joint arm_camera_mount_joint: origin xyz=0.025 0.0 0.08 rpy=0 0 0 -> xyz=0.025 -0.060 0.08 rpy=0 0 0

File: src/hoverboard_base/urdf/robot_piper.urdf.xacro (robot description, xacro)
@@ -723,5 +723,6 @@
     <parent link="gripper_base"/>
     <child link="arm_camera_link"/>
-    <origin xyz="0.025 0.0 0.08" rpy="0 0 0"/>
+    <!-- Camara del brazo desfasada 6 cm a la derecha (-0.06 m en eje Y) respecto al centro de la pinza -->
+    <origin xyz="0.025 -0.060 0.08" rpy="0 0 0"/>
   </joint>
   <!-- Marco Óptico Orbbec DaBai (Estándar ROS: Z adelante, X derecha, Y abajo) -->
