Commit message: feat(manipulation): center wrist camera offset to 0.0m in URDF, YAML and kinematics

File: src/hoverboard_base/urdf/robot.urdf (robot description, URDF)
Before this commit: robot robot_athome, 28 links, 27 joints
Joints:
- joint arm_camera_mount_joint: origin xyz=0.025 -0.060 0.08 rpy=0 0 0 -> xyz=0.025 0.0 0.08 rpy=0 0 0
- joint joint7: limit lower=0 upper=0.035 effort=10 velocity=1 -> lower=0 upper=0.0525 effort=10 velocity=1
- joint joint8: limit lower=-0.035 upper=0 effort=10 velocity=1 -> lower=-0.0525 upper=0 effort=10 velocity=1

File: src/hoverboard_base/urdf/robot_piper.urdf.xacro (robot description, xacro)
@@ -669,5 +669,5 @@
     <child link="link7" />
     <axis xyz="0 0 1" />
-    <limit lower="0" upper="0.035" effort="10" velocity="1" />
+    <limit lower="0" upper="0.0525" effort="10" velocity="1" />
   </joint>
   <!-- Dedo Derecho Pinza (Joint 8 - Prismático) -->
@@ -697,5 +697,5 @@
     <child link="link8" />
     <axis xyz="0 0 -1" />
-    <limit lower="-0.035" upper="0" effort="10" velocity="1" />
+    <limit lower="-0.0525" upper="0" effort="10" velocity="1" />
   </joint>
   <!-- Cámara de Muñeca Orbbec DaBai DC1 (Eye-in-Hand) -->
@@ -723,6 +723,6 @@
     <parent link="gripper_base"/>
     <child link="arm_camera_link"/>
-    <!-- Camara del brazo desfasada 6 cm a la derecha (-0.06 m en eje Y) respecto al centro de la pinza -->
-    <origin xyz="0.025 -0.060 0.08" rpy="0 0 0"/>
+    <!-- Camara del brazo centrada (0.0 m en eje Y) respecto al centro de la pinza -->
+    <origin xyz="0.025 0.0 0.08" rpy="0 0 0"/>
   </joint>
   <!-- Marco Óptico Orbbec DaBai (Estándar ROS: Z adelante, X derecha, Y abajo) -->

Commit message: feat(manipulacion): simplify manipulation from scratch with camera 8cm back and single distance adjustment

File: src/hoverboard_base/urdf/robot.urdf (robot description, URDF)
Before this commit: robot robot_athome, 28 links, 27 joints
Joints:
- joint arm_camera_mount_joint: origin xyz=0.025 0.0 0.08 rpy=0 0 0 -> xyz=0.025 0.0 0.00 rpy=0 0 0

File: src/hoverboard_base/urdf/robot_piper.urdf.xacro (robot description, xacro)
@@ -723,6 +723,6 @@
     <parent link="gripper_base"/>
     <child link="arm_camera_link"/>
-    <!-- Camara del brazo centrada (0.0 m en eje Y) respecto al centro de la pinza -->
-    <origin xyz="0.025 0.0 0.08" rpy="0 0 0"/>
+    <!-- Camara del brazo montada 8cm hacia atras y perfectamente centrada (y=0.0) -->
+    <origin xyz="0.025 0.0 0.00" rpy="0 0 0"/>
   </joint>
   <!-- Marco Óptico Orbbec DaBai (Estándar ROS: Z adelante, X derecha, Y abajo) -->

Commit message: feat: add ArUco detection priority, prismatic torso lift with calibrated NEMA 23 limits and move arm 15cm back

File: src/hoverboard_base/urdf/robot.urdf (robot description, URDF)
Before this commit: robot robot_athome, 28 links, 27 joints
Links:
- link torso_column: geometry collision box size=0.08 0.08 1.3; visual box size=0.06 0.06 1.3
Joints:
- joint cube_to_arm_joint: origin xyz=0.0 0.175 0.10 rpy=-1.5707963 0 0 -> xyz=-0.15 0.175 0.10 rpy=-1.5707963 0 0
- joint torso_lift_joint: axis (none) -> 0 0 1; limit (none) -> lower=-0.75 upper=0.0 effort=500.0 velocity=0.10; origin xyz=0 0 1.0 rpy=0 0 0 -> xyz=0 0 1.26 rpy=0 0 0; type fixed -> prismatic

File: src/hoverboard_base/urdf/robot_piper.urdf.xacro (robot description, xacro)
@@ -18,8 +18,8 @@
   <xacro:property name="laser_offset_y" value="0.00"/>
   <xacro:property name="laser_offset_z" value="0.18"/>
-  <!-- Sistema de Elevación Torso / Columna (Exactamente en el medio de la base, 1.0 m altura) -->
+  <!-- Sistema de Elevación Torso / Columna (Exactamente en el medio de la base, 1.30 m altura) -->
   <xacro:property name="column_x"               value="0.0"/>
   <xacro:property name="column_y"               value="0.0"/>
-  <xacro:property name="column_height"          value="1.0"/>
+  <xacro:property name="column_height"          value="1.30"/>
   <xacro:property name="column_width"           value="0.06"/>
   <xacro:property name="column_collision_width" value="0.08"/>
@@ -28,4 +28,11 @@
   <xacro:property name="carriage_width"         value="0.38"/>
   <xacro:property name="carriage_height"        value="0.02"/>
+  <!-- Parámetros del Eje Z (Motor NEMA 23 y fines de carrera) -->
+  <!-- Fin de carrera superior: cara inferior del cubo a exactamente 1.00 m del piso -->
+  <!-- Fin de carrera inferior: cara inferior del cubo a exactamente 0.40 m del piso (carrera de trabajo: 0.60 m) -->
+  <!-- Carrera mecánica máxima hasta el piso: ~0.75 m -->
+  <xacro:property name="torso_lift_top_z"       value="1.26"/>
+  <xacro:property name="torso_switch_stroke"    value="0.60"/>
+  <xacro:property name="torso_floor_stroke"     value="0.75"/>
   <!-- Prisma Estructural del Torso de Subir y Bajar (35 cm ancho x 25 cm profundidad x 35 cm alto) -->
   <xacro:property name="prism_size_x"           value="0.25"/> <!-- 25 cm hacia adelante desde la pared frontal del elevador -->
@@ -229,8 +236,15 @@
     </inertial>
   </link>
-  <joint name="torso_lift_joint" type="fixed">
+  <!-- Articulación prismática de elevación del torso controlada por NEMA 23 -->
+  <!-- Posición 0.0 m = Fin de carrera superior (cara inferior del cubo a exactamente 1.00 m del piso) -->
+  <!-- Posición -0.60 m = Fin de carrera inferior (cara inferior del cubo a exactamente 0.40 m del piso) -->
+  <!-- Posición -0.75 m = Descenso máximo hacia el piso (~75 cm) para manipular objetos en el suelo -->
+  <joint name="torso_lift_joint" type="prismatic">
     <parent link="torso_column"/>
     <child link="torso_lift_link"/>
-    <origin xyz="0 0 ${column_height}" rpy="0 0 0"/>
+    <axis xyz="0 0 1"/>
+    <origin xyz="0 0 ${torso_lift_top_z}" rpy="0 0 0"/>
+    <limit lower="-${torso_floor_stroke}" upper="0.0" effort="500.0" velocity="0.10"/>
+    <dynamics damping="10.0" friction="5.0"/>
   </joint>
   <!-- ==================== PRISMA ESTRUCTURAL DEL TORSO (SUBIR Y BAJAR) ==================== -->
@@ -436,9 +450,9 @@
     </collision>
   </link>
-  <!-- Montaje sobre el lado lateral izquierdo del prisma del torso, como un brazo humano en el hombro -->
+  <!-- Montaje sobre el lado lateral izquierdo del prisma del torso, retrasado 15 cm hacia atrás -->
   <joint name="cube_to_arm_joint" type="fixed">
     <parent link="mounting_cube_link"/>
     <child link="arm_base_link"/>
-    <origin xyz="0.0 ${prism_size_y / 2.0} 0.10" rpy="-1.5707963 0 0"/>
+    <origin xyz="-0.15 ${prism_size_y / 2.0} 0.10" rpy="-1.5707963 0 0"/>
   </joint>
   <!-- Link 1 (Joint 1 - Rotación en Z) -->

Commit message: Calibracion de altura y URDF con medidas reales: mesa a 76cm, gripper a 85cm, hombro a 1.065m

File: src/hoverboard_base/urdf/robot.urdf (robot description, URDF)
Before this commit: robot robot_athome, 28 links, 27 joints
Joints:
- joint cube_to_arm_joint: origin xyz=-0.15 0.175 0.10 rpy=-1.5707963 0 0 -> xyz=-0.15 0.175 -0.11 rpy=-1.5707963 0 0

File: src/hoverboard_base/urdf/robot_piper.urdf.xacro (robot description, xacro)
@@ -450,9 +450,9 @@
     </collision>
   </link>
-  <!-- Montaje sobre el lado lateral izquierdo del prisma del torso, retrasado 15 cm hacia atrás -->
+  <!-- Montaje sobre el lado lateral izquierdo del prisma del torso, retrasado 15 cm hacia atrás y calibrado a 85 cm de altura del gripper -->
   <joint name="cube_to_arm_joint" type="fixed">
     <parent link="mounting_cube_link"/>
     <child link="arm_base_link"/>
-    <origin xyz="-0.15 ${prism_size_y / 2.0} 0.10" rpy="-1.5707963 0 0"/>
+    <origin xyz="-0.15 ${prism_size_y / 2.0} -0.11" rpy="-1.5707963 0 0"/>
   </joint>
   <!-- Link 1 (Joint 1 - Rotación en Z) -->

Commit message: feat(hri): Implement RoboCup @Home Receptionist Challenge node and update ZED Mini offsets

File: src/hoverboard_base/urdf/robot.urdf (robot description, URDF)
Before this commit: robot robot_athome, 28 links, 27 joints
Links:
- added link zed_camera_link
- added link zed_left_camera_frame
- added link zed_left_camera_optical_frame
- added link zed_right_camera_frame
- added link zed_right_camera_optical_frame
- link camera_link: mass 0.072 -> 0.063; geometry collision box size=0.0305 0.1245 0.0305; visual box size=0.0305 0.1245 0.0305
Joints:
- added joint zed_camera_link_joint: type fixed, parent camera_link, child zed_camera_link, origin xyz=0 0 0 rpy=0 0 0
- added joint zed_left_camera_joint: type fixed, parent camera_link, child zed_left_camera_frame, origin xyz=0 0.0315 0 rpy=0 0 0
- added joint zed_left_camera_optical_joint: type fixed, parent zed_left_camera_frame, child zed_left_camera_optical_frame, origin xyz=0 0 0 rpy=-1.5707963 0 -1.5707963
- added joint zed_right_camera_joint: type fixed, parent camera_link, child zed_right_camera_frame, origin xyz=0 -0.0315 0 rpy=0 0 0
- added joint zed_right_camera_optical_joint: type fixed, parent zed_right_camera_frame, child zed_right_camera_optical_frame, origin xyz=0 0 0 rpy=-1.5707963 0 -1.5707963
- joint camera_color_optical_joint: origin xyz=0 0 0 rpy=-1.5707963 0 -1.5707963 -> xyz=0 0 0 rpy=0 0 0; parent camera_link -> zed_left_camera_optical_frame
- joint camera_mount_joint: origin xyz=0.035 0.0 0.015 rpy=0 0 0 -> xyz=0.135 0.0 0.015 rpy=0 0 0

File: src/hoverboard_base/urdf/robot_piper.urdf.xacro (robot description, xacro)
@@ -92,4 +92,7 @@
     <color rgba="0.08 0.08 0.08 1.0"/>
   </material>
+  <material name="zed_black">
+    <color rgba="0.12 0.12 0.12 1.0"/>
+  </material>
   <!-- ==================== BASE FOOTPRINT ==================== -->
   <link name="base_footprint"/>
@@ -395,36 +398,71 @@
     <limit lower="-0.7854" upper="0.7854" effort="2.5" velocity="3.14"/>
   </joint>
-  <!-- Cámara RealSense D435 en Cabezal -->
+  <!-- Cámara Estereoscópica Stereolabs ZED Mini en Cabezal Pan-Tilt -->
+  <!-- Desplazada 10 cm adicionales hacia adelante respecto al anclaje anterior (x = 0.135 m) -->
   <joint name="camera_mount_joint" type="fixed">
     <parent link="tilt_link"/>
     <child link="camera_link"/>
-    <origin xyz="0.035 0.0 0.015" rpy="0 0 0"/>
-  </joint>
+    <origin xyz="0.135 0.0 0.015" rpy="0 0 0"/>
+  </joint>
+  <!-- Chasis Central de la ZED Mini (124.5 mm ancho x 30.5 mm prof x 30.5 mm alto, peso ~63g) -->
   <link name="camera_link">
     <visual>
       <origin xyz="0 0 0" rpy="0 0 0"/>
       <geometry>
-        <box size="0.025 0.090 0.025"/>
-      </geometry>
-      <material name="realsense_silver"/>
-    </visual>
-    <collision>
-      <origin xyz="0 0 0" rpy="0 0 0"/>
-      <geometry>
-        <box size="0.025 0.090 0.025"/>
-      </geometry>
-    </collision>
-    <inertial>
-      <origin xyz="0 0 0" rpy="0 0 0"/>
-      <mass value="0.072"/>
-      <inertia ixx="0.00005" ixy="0.0" ixz="0.0" iyy="0.00001" iyz="0.0" izz="0.00005"/>
-    </inertial>
-  </link>
-  <!-- Marco Óptico RealSense (Estándar ROS: Z adelante, X derecha, Y abajo) -->
+        <box size="0.0305 0.1245 0.0305"/>
+      </geometry>
+      <material name="zed_black"/>
+    </visual>
+    <collision>
+      <origin xyz="0 0 0" rpy="0 0 0"/>
+      <geometry>
+        <box size="0.0305 0.1245 0.0305"/>
+      </geometry>
+    </collision>
+    <inertial>
+      <origin xyz="0 0 0" rpy="0 0 0"/>
+      <mass value="0.063"/>
+      <inertia ixx="0.00008" ixy="0.0" ixz="0.0" iyy="0.00001" iyz="0.0" izz="0.00008"/>
+    </inertial>
+  </link>
+  <!-- Enlace zed_camera_link para compatibilidad nativa con el wrapper oficial de Stereolabs -->
+  <link name="zed_camera_link"/>
+  <joint name="zed_camera_link_joint" type="fixed">
+    <parent link="camera_link"/>
+    <child link="zed_camera_link"/>
+    <origin xyz="0 0 0" rpy="0 0 0"/>
+  </joint>
+  <!-- Lente Izquierda ZED Mini (Baseline 63 mm -> +31.5 mm en Y) -->
+  <link name="zed_left_camera_frame"/>
+  <joint name="zed_left_camera_joint" type="fixed">
+    <parent link="camera_link"/>
+    <child link="zed_left_camera_frame"/>
+    <origin xyz="0 0.0315 0" rpy="0 0 0"/>
+  </joint>
+  <link name="zed_left_camera_optical_frame"/>
+  <joint name="zed_left_camera_optical_joint" type="fixed">
+    <parent link="zed_left_camera_frame"/>
+    <child link="zed_left_camera_optical_frame"/>
+    <origin xyz="0 0 0" rpy="-1.5707963 0 -1.5707963"/>
+  </joint>
+  <!-- Lente Derecha ZED Mini (Baseline 63 mm -> -31.5 mm en Y) -->
+  <link name="zed_right_camera_frame"/>
+  <joint name="zed_right_camera_joint" type="fixed">
+    <parent link="camera_link"/>
+    <child link="zed_right_camera_frame"/>
+    <origin xyz="0 -0.0315 0" rpy="0 0 0"/>
+  </joint>
+  <link name="zed_right_camera_optical_frame"/>
+  <joint name="zed_right_camera_optical_joint" type="fixed">
+    <parent link="zed_right_camera_frame"/>
+    <child link="zed_right_camera_optical_frame"/>
+    <origin xyz="0 0 0" rpy="-1.5707963 0 -1.5707963"/>
+  </joint>
+  <!-- Marco Óptico de Color (Mantenido para 100% de retrocompatibilidad con nodos de visión y RViz) -->
   <link name="camera_color_optical_frame"/>
   <joint name="camera_color_optical_joint" type="fixed">
-    <parent link="camera_link"/>
+    <parent link="zed_left_camera_optical_frame"/>
     <child link="camera_color_optical_frame"/>
-    <origin xyz="0 0 0" rpy="-1.5707963 0 -1.5707963"/>
+    <origin xyz="0 0 0" rpy="0 0 0"/>
   </joint>
   <!-- ==================== BRAZO ROBÓTICO AGILEX PIPER 6-DOF ==================== -->
