Commit message: feat(hri): adapt fbot_hri architecture, RealSense D435 integration, URDF modularization and mic anti-echo

File: src/hoverboard_base/urdf/robot.urdf (robot description, URDF)
Before this commit: robot robot_athome, 33 links, 32 joints
Links:
- removed link zed_camera_link
- removed link zed_left_camera_frame
- removed link zed_left_camera_optical_frame
- removed link zed_right_camera_frame
- removed link zed_right_camera_optical_frame
- added link camera_color_frame
- added link camera_depth_frame
- added link camera_depth_optical_frame
- link camera_link: mass 0.063 -> 0.072; geometry collision box size=0.025 0.090 0.025; visual box size=0.025 0.090 0.025
Joints:
- removed joint zed_camera_link_joint
- removed joint zed_left_camera_joint
- removed joint zed_left_camera_optical_joint
- removed joint zed_right_camera_joint
- removed joint zed_right_camera_optical_joint
- added joint camera_color_joint: type fixed, parent camera_link, child camera_color_frame, origin xyz=1.4876e-05 0.015106 -9.367e-05 rpy=0.016168 0.002748 -0.007364
- added joint camera_depth_joint: type fixed, parent camera_link, child camera_depth_frame, origin xyz=0 0 0 rpy=0 0 0
- added joint camera_depth_optical_joint: type fixed, parent camera_depth_frame, child camera_depth_optical_frame, origin xyz=0 0 0 rpy=-1.5707963 0 -1.5707963
- joint camera_color_optical_joint: origin xyz=0 0 0 rpy=0 0 0 -> xyz=0 0 0 rpy=-1.5707963 0 -1.5707963; parent zed_left_camera_optical_frame -> camera_color_frame

File: src/hoverboard_base/urdf/robot.urdf.xacro (robot description, xacro)
@@ -1,282 +1,13 @@
 <?xml version="1.0"?>
-<robot xmlns:xacro="http://www.ros.org/wiki/xacro" name="hoverboard_robot">
-  <!-- ==================== PROPIEDADES CONFIGURABLES ==================== -->
-  <xacro:property name="chassis_length" value="0.48"/>
-  <xacro:property name="chassis_width"  value="0.48"/>
-  <xacro:property name="chassis_height" value="0.05"/>
-  <xacro:property name="ground_clearance" value="0.04"/>
-  <!-- Distancia efectiva calibrada entre ruedas: 56.20 cm -> offset Y = +/- 0.281m -->
-  <xacro:property name="track_width"    value="0.5620"/>
-  <xacro:property name="wheel_radius"   value="0.0853"/>
-  <xacro:property name="wheel_width"    value="0.055"/>
-  <xacro:property name="wheel_offset_x" value="0.095"/>
-  <!-- Rueda loca trasera -->
-  <xacro:property name="caster_offset_x" value="-0.20"/>
-  <xacro:property name="caster_radius"   value="0.04"/>
-  <!-- Sensor LiDAR Hokuyo -->
-  <xacro:property name="laser_offset_x" value="0.22"/>
-  <xacro:property name="laser_offset_y" value="0.00"/>
-  <xacro:property name="laser_offset_z" value="0.18"/>
-  <!-- Sistema de Elevación Torso / Columna (Exactamente en el medio de la base, 1.0 m altura) -->
-  <xacro:property name="column_x"       value="0.0"/>
-  <xacro:property name="column_y"       value="0.0"/>
-  <xacro:property name="column_height"  value="1.0"/>
-  <xacro:property name="column_width"   value="0.06"/>
-  <!-- ==================== MATERIALES ==================== -->
-  <material name="chassis_blue">
-    <color rgba="0.15 0.45 0.85 0.95"/>
-  </material>
-  <material name="wheel_black">
-    <color rgba="0.10 0.10 0.10 1.0"/>
-  </material>
-  <material name="laser_red">
-    <color rgba="0.90 0.10 0.10 1.0"/>
-  </material>
-  <material name="caster_gray">
-    <color rgba="0.35 0.35 0.35 1.0"/>
-  </material>
-  <material name="column_aluminum">
-    <color rgba="0.65 0.65 0.70 1.0"/>
-  </material>
-  <material name="pantilt_dark">
-    <color rgba="0.18 0.18 0.18 1.0"/>
-  </material>
-  <material name="realsense_silver">
-    <color rgba="0.75 0.75 0.75 1.0"/>
-  </material>
-  <!-- ==================== BASE FOOTPRINT ==================== -->
-  <link name="base_footprint"/>
-  <!-- ==================== CHASIS ==================== -->
-  <link name="base_link">
-    <visual>
-      <origin xyz="0 0 ${ground_clearance + chassis_height / 2.0}" rpy="0 0 0"/>
-      <geometry>
-        <box size="${chassis_length} ${chassis_width} ${chassis_height}"/>
-      </geometry>
-      <material name="chassis_blue"/>
-    </visual>
-    <collision>
-      <origin xyz="0 0 ${ground_clearance + chassis_height / 2.0}" rpy="0 0 0"/>
-      <geometry>
-        <box size="${chassis_length} ${chassis_width} ${chassis_height}"/>
-      </geometry>
-    </collision>
-    <inertial>
-      <origin xyz="0 0 ${ground_clearance + chassis_height / 2.0}" rpy="0 0 0"/>
-      <mass value="12.0"/>
-      <inertia ixx="0.233" ixy="0.0" ixz="0.0" iyy="0.233" iyz="0.0" izz="0.461"/>
-    </inertial>
-  </link>
-  <joint name="base_joint" type="fixed">
-    <parent link="base_footprint"/>
-    <child link="base_link"/>
-    <origin xyz="0 0 0" rpy="0 0 0"/>
-  </joint>
-  <!-- Macro para ruedas -->
-  <xacro:macro name="hover_wheel" params="prefix y_reflect">
-    <link name="${prefix}_wheel">
-      <visual>
-        <origin xyz="0 0 0" rpy="1.5707963 0 0"/>
-        <geometry>
-          <cylinder radius="${wheel_radius}" length="${wheel_width}"/>
-        </geometry>
-        <material name="wheel_black"/>
-      </visual>
-      <collision>
-        <origin xyz="0 0 0" rpy="1.5707963 0 0"/>
-        <geometry>
-          <cylinder radius="${wheel_radius}" length="${wheel_width}"/>
-        </geometry>
-      </collision>
-    </link>
-    <joint name="${prefix}_wheel_joint" type="continuous">
-      <parent link="base_link"/>
-      <child link="${prefix}_wheel"/>
-      <origin xyz="${wheel_offset_x} ${y_reflect * track_width / 2.0} ${wheel_radius}" rpy="0 0 0"/>
-      <axis xyz="0 1 0"/>
-    </joint>
-  </xacro:macro>
-  <xacro:hover_wheel prefix="left" y_reflect="1"/>
-  <xacro:hover_wheel prefix="right" y_reflect="-1"/>
-  <!-- Rueda loca trasera -->
-  <link name="rear_caster">
-    <visual>
-      <origin xyz="0 0 0" rpy="0 0 0"/>
-      <geometry>
-        <sphere radius="${caster_radius}"/>
-      </geometry>
-      <material name="caster_gray"/>
-    </visual>
-    <collision>
-      <origin xyz="0 0 0" rpy="0 0 0"/>
-      <geometry>
-        <sphere radius="${caster_radius}"/>
-      </geometry>
-    </collision>
-  </link>
-  <joint name="rear_caster_joint" type="fixed">
-    <parent link="base_link"/>
-    <child link="rear_caster"/>
-    <origin xyz="${caster_offset_x} 0.0 ${caster_radius}" rpy="0 0 0"/>
-  </joint>
-  <!-- LiDAR Hokuyo -->
-  <link name="laser">
-    <visual>
-      <origin xyz="0 0 0" rpy="0 0 0"/>
-      <geometry>
-        <cylinder radius="0.035" length="0.05"/>
-      </geometry>
-      <material name="laser_red"/>
-    </visual>
-    <collision>
-      <origin xyz="0 0 0" rpy="0 0 0"/>
-      <geometry>
-        <cylinder radius="0.035" length="0.05"/>
-      </geometry>
-    </collision>
-  </link>
-  <joint name="laser_joint" type="fixed">
-    <parent link="base_link"/>
-    <child link="laser"/>
-    <origin xyz="${laser_offset_x} ${laser_offset_y} ${laser_offset_z}" rpy="0 0 0"/>
-  </joint>
-  <!-- ==================== SISTEMA DE SUBIR Y BAJAR (TORSO VERTICAL) ==================== -->
-  <!-- Columna estructural fija exactamente en el medio de la base (x=0, y=0) con 1 metro de altura -->
-  <link name="torso_column">
-    <visual>
-      <origin xyz="0 0 ${column_height / 2.0}" rpy="0 0 0"/>
-      <geometry>
-        <box size="${column_width} ${column_width} ${column_height}"/>
-      </geometry>
-      <material name="column_aluminum"/>
-    </visual>
-    <collision>
-      <origin xyz="0 0 ${column_height / 2.0}" rpy="0 0 0"/>
-      <geometry>
-        <box size="${column_width} ${column_width} ${column_height}"/>
-      </geometry>
-    </collision>
-    <inertial>
-      <origin xyz="0 0 ${column_height / 2.0}" rpy="0 0 0"/>
-      <mass value="3.5"/>
-      <inertia ixx="0.292" ixy="0.0" ixz="0.0" iyy="0.292" iyz="0.0" izz="0.002"/>
-    </inertial>
-  </link>
-  <joint name="torso_column_joint" type="fixed">
-    <parent link="base_link"/>
-    <child link="torso_column"/>
-    <origin xyz="${column_x} ${column_y} ${ground_clearance + chassis_height}" rpy="0 0 0"/>
-  </joint>
-  <!-- Plataforma superior móvil del elevador (a 1.0 m arriba en la parte superior) -->
-  <link name="torso_lift_link">
-    <visual>
-      <origin xyz="0 0 0" rpy="0 0 0"/>
-      <geometry>
-        <box size="0.10 0.12 0.02"/>
-      </geometry>
-      <material name="pantilt_dark"/>
-    </visual>
-    <collision>
-      <origin xyz="0 0 0" rpy="0 0 0"/>
-      <geometry>
-        <box size="0.10 0.12 0.02"/>
-      </geometry>
-    </collision>
-  </link>
-  <!-- Joint de elevación / tope superior de columna (fijo a 1.0 m de altura) -->
-  <joint name="torso_lift_joint" type="fixed">
-    <parent link="torso_column"/>
-    <child link="torso_lift_link"/>
-    <origin xyz="0 0 ${column_height}" rpy="0 0 0"/>
-  </joint>
-  <!-- ==================== SISTEMA PAN-TILT ==================== -->
-  <!-- Base de montaje del Pan-Tilt -->
-  <link name="pan_tilt_base_link">
-    <visual>
-      <origin xyz="0 0 0.015" rpy="0 0 0"/>
-      <geometry>
-        <cylinder radius="0.035" length="0.03"/>
-      </geometry>
-      <material name="pantilt_dark"/>
-    </visual>
-    <collision>
-      <origin xyz="0 0 0.015" rpy="0 0 0"/>
-      <geometry>
-        <cylinder radius="0.035" length="0.03"/>
-      </geometry>
-    </collision>
-  </link>
-  <joint name="pan_tilt_base_joint" type="fixed">
-    <parent link="torso_lift_link"/>
-    <child link="pan_tilt_base_link"/>
-    <origin xyz="0 0 0.01" rpy="0 0 0"/>
-  </joint>
-  <!-- Motor 1: Pan Joint (Giro Horizontal en Z) -->
-  <link name="pan_link">
-    <visual>
-      <origin xyz="0 0 0.025" rpy="0 0 0"/>
-      <geometry>
-        <box size="0.045 0.045 0.05"/>
-      </geometry>
-      <material name="pantilt_dark"/>
-    </visual>
-    <collision>
-      <origin xyz="0 0 0.025" rpy="0 0 0"/>
-      <geometry>
-        <box size="0.045 0.045 0.05"/>
-      </geometry>
-    </collision>
-  </link>
-  <joint name="pan_joint" type="revolute">
-    <parent link="pan_tilt_base_link"/>
-    <child link="pan_link"/>
-    <origin xyz="0 0 0.03" rpy="0 0 0"/>
-    <axis xyz="0 0 1"/>
-    <limit lower="-1.5708" upper="1.5708" effort="2.5" velocity="3.14"/>
-  </joint>
-  <!-- Motor 2: Tilt Joint (Inclinación Vertical en Y) -->
-  <link name="tilt_link">
-    <visual>
-      <origin xyz="0.015 0 0.01" rpy="0 0 0"/>
-      <geometry>
-        <box size="0.04 0.10 0.03"/>
-      </geometry>
-      <material name="pantilt_dark"/>
-    </visual>
-    <collision>
-      <origin xyz="0.015 0 0.01" rpy="0 0 0"/>
-      <geometry>
-        <box size="0.04 0.10 0.03"/>
-      </geometry>
-    </collision>
-  </link>
-  <joint name="tilt_joint" type="revolute">
-    <parent link="pan_link"/>
-    <child link="tilt_link"/>
-    <origin xyz="0 0 0.05" rpy="0 0 0"/>
-    <axis xyz="0 1 0"/>
-    <limit lower="-0.7854" upper="0.7854" effort="2.5" velocity="3.14"/>
-  </joint>
-  <!-- ==================== CÁMARA INTEL REALSENSE D435 ==================== -->
-  <!-- Conexión rígida entre el soporte tilt y el marco base de la RealSense (camera_link) -->
-  <joint name="camera_mount_joint" type="fixed">
-    <parent link="tilt_link"/>
-    <child link="camera_link"/>
-    <origin xyz="0.035 0.0 0.015" rpy="0 0 0"/>
-  </joint>
-  <link name="camera_link">
-    <visual>
-      <origin xyz="0 0 0" rpy="0 0 0"/>
-      <geometry>
-        <box size="0.025 0.090 0.025"/>
-      </geometry>
-      <material name="realsense_silver"/>
-    </visual>
-    <collision>
-      <origin xyz="0 0 0" rpy="0 0 0"/>
-      <geometry>
-        <box size="0.025 0.090 0.025"/>
-      </geometry>
-    </collision>
-  </link>
+<!-- Robot RoboCup @Home (base hoverboard + torso elevador + pan-tilt con RealSense D435 + brazo Piper).
+     Archivo principal: solo incluye los modulos. Las rutas son relativas a este archivo.
+     Compilar con scripts/build_urdf.sh (genera robot.urdf, que es el que cargan los launch). -->
+<robot xmlns:xacro="http://www.ros.org/wiki/xacro" name="robot_athome">
+  <!-- properties.xacro va PRIMERO: sus propiedades deben ser visibles en los demas modulos -->
+  <xacro:include filename="xacro/properties.xacro"/>
+  <xacro:include filename="xacro/materials.xacro"/>
+  <xacro:include filename="xacro/base.xacro"/>
+  <xacro:include filename="xacro/torso.xacro"/>
+  <xacro:include filename="xacro/head.xacro"/>
+  <xacro:include filename="xacro/arm_piper.xacro"/>
 </robot>
